File: subassembly/encoder/rotary_input_board/rotary_input_board.kicad_sch (KiCad schematic)
At the start: 48 parts, among them J1 Conn_01x05, J3 SOICbite-SWD, J4 Conn_01x05, U1 ATSAMD10D13A-M

Commit message: Before firmware normalization
Other:
- note added: "Resistor Values: Blue: 3.2V - 5 ohm Red: 2.0V - 65 ohm Green: 2.0V - 65 ohm"
Changed lines of the file:
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@@
+    (effects (font (size 1.27 1.27)) (justify left bottom))
+  )
+  (text "Resistor Values:\nBlue: 3.2V - 5 ohm\nRed: 2.0V - 65 ohm\nGreen: 2.0V - 65 ohm"
+    (at 171.45 45.085 0)
     (effects (font (size 1.27 1.27)) (justify left bottom))
   )
